File: disco_tft_adapter.kicad_sch (KiCad schematic)
At the start: 21 parts, among them J1 QTH-030-02-L-D-A, J2 F31L-1A7H1-11030

Commit message: [project] ready up for production, added more infos for bom
Parts:
- C1, C2, C3, C5, C8: Mouser Part Number (none) -> 603-C0603MRY5V9BB104
- C4, C6, C9: Mouser Part Number (none) -> 581-08055D475KAT2A
- C7: Mouser Part Number (none) -> 603-CC805KKX5R9BB225
- L1: Mouser Part Number (none) -> 994-LPS4018-103MRC
- R1, R2: Mouser Part Number (none) -> 71-RCA06030000ZSEASR
- R3: Mouser Part Number (none) -> 71-CRCW12065R10FKEA
Changed lines of the file:
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@@
 			)
 		)
+		(property "Mouser Part Number" "603-C0603MRY5V9BB104"
+			(at 39.37 162.56 0)
+			(effects
+				(font
+					(size 1.27 1.27)
+				)
+				(hide yes)
+			)
+		)
 		(pin "2"
 		)
@@
 			)
 		)
+		(property "Mouser Part Number" "603-CC805KKX5R9BB225"
+			(at 241.3 39.37 0)
+			(effects
+				(font
+					(size 1.27 1.27)
+				)
+				(hide yes)
+			)
+		)
 		(pin "2"
 		)
@@
 			)
 		)
+		(property "Mouser Part Number" "994-LPS4018-103MRC"
+			(at 205.74 34.29 90)
+			(effects
+				(font
+					(size 1.27 1.27)
+				)
+				(hide yes)
+			)
+		)
 		(pin "1"
 		)
@@
 			)
 		)
+		(property "Mouser Part Number" "581-08055D475KAT2A"
+			(at 104.14 162.56 0)
+			(effects
+				(font
+					(size 1.27 1.27)
+				)
+				(hide yes)
+			)
+		)
 		(pin "2"
 		)
@@
 			)
 		)
+		(property "Mouser Part Number" "603-C0603MRY5V9BB104"
+			(at 25.4 162.56 0)
+			(effects
+				(font
+					(size 1.27 1.27)
+				)
+				(hide yes)
+			)
+		)
 		(pin "2"
 		)
@@
 			)
 		)
+		(property "Mouser Part Number" "71-RCA06030000ZSEASR"
+			(at 172.72 34.29 0)
+			(effects
+				(font
+					(size 1.27 1.27)
+				)
+				(hide yes)
+			)
+		)
 		(pin "2"
 		)
@@
 			)
 		)
+		(property "Mouser Part Number" "603-C0603MRY5V9BB104"
+			(at 173.99 58.42 0)
+			(effects
+				(font
+					(size 1.27 1.27)
+				)
+				(hide yes)
+			)
+		)
 		(pin "2"
 		)
@@
 			)
 		)
+		(property "Mouser Part Number" "581-08055D475KAT2A"
+			(at 186.69 58.42 0)
+			(effects
+				(font
+					(size 1.27 1.27)
+				)
+				(hide yes)
+			)
+		)
 		(pin "2"
 		)
@@
 			)
 		)
+		(property "Mouser Part Number" "71-RCA06030000ZSEASR"
+			(at 180.34 34.29 0)
+			(effects
+				(font
+					(size 1.27 1.27)
+				)
+				(hide yes)
+			)
+		)
 		(pin "2"
 		)
@@
 			)
 		)
+		(property "Mouser Part Number" "581-08055D475KAT2A"
+			(at 76.2 162.56 0)
+			(effects
+				(font
+					(size 1.27 1.27)
+				)
+				(hide yes)
+			)
+		)
 		(pin "2"
 		)
@@
 			)
 		)
+		(property "Mouser Part Number" "603-C0603MRY5V9BB104"
+			(at 90.17 162.56 0)
+			(effects
+				(font
+					(size 1.27 1.27)
+				)
+				(hide yes)
+			)
+		)
 		(pin "2"
 		)
@@
 			)
 		)
+		(property "Mouser Part Number" "603-C0603MRY5V9BB104"
+			(at 62.23 162.56 0)
+			(effects
+				(font
+					(size 1.27 1.27)
+				)
+				(hide yes)
+			)
+		)
 		(pin "2"
 		)
@@
 			(at 229.87 59.69 0)
 			(effects
+				(font
+					(size 1.27 1.27)
+				)
+				(hide yes)
+			)
+		)
+		(property "Mouser Part Number" "71-CRCW12065R10FKEA"
+			(at 229.87 59.69 0)
+			(effects
